Commit message: try to run control_manager FAILED

File: stiu_setup_tf/urdf/stiu.xacro (robot description, xacro)
@@ -23,5 +23,5 @@
 		<visual>
 			<geometry>
-				<box size = "0.11 0.174 0.06"/>
+				<box size = "0.174 0.11 0.06"/>
 			</geometry>
 			<material name="blue">
@@ -31,5 +31,5 @@
 		<collision>
 			<geometry>
-				<box size = "0.11 0.174 0.06"/>
+				<box size = "0.174 0.11 0.06"/>
 			</geometry>
 		</collision>
@@ -57,8 +57,30 @@
 			<parent link="base_link"/>
 			<child link="${prefix}_wheel"/>
-			<origin xyz="${0.05*reflect} 0 -0.03" rpy="0 ${pi/2} 0"/>
+			<origin xyz="0 ${0.05*reflect} -0.03" rpy="${pi/2} 0 0"/>
       			<limit effort="100" velocity="100" />
 			<joint_properties damping="0.0" friction="0.0" />
 		</joint>
+		<gazebo reference="${prefix}_wheel">
+			<mu1 value="200.0"/>
+			<mu2 value="100.0"/>
+			<kp value="10000000.0"/>
+			<kd value="1.0"/>
+			<material>Gazebo/Grey</material>
+		</gazebo>
+		<gazebo>
+			<plugin name="gazebo_ros_control" filename="libgazebo_ros_control.so">
+  			</plugin>
+		</gazebo>
+		<!-- This block connects the wheel joint to an actuator (motor), which informs both
+    		simulation and visualization of the robot -->
+		<!-- <transmission name="${prefix}_wheel_trans" type="SimpleTransmission">
+      			<type>transmission_interface/SimpleTransmission</type>
+      			<actuator name="${prefix}_wheel_motor">
+        			<mechanicalReduction>1</mechanicalReduction>
+      			</actuator>
+			<joint name="${prefix}_wheel_joint">
+        			<hardwareInterface>VelocityJointInterface</hardwareInterface>
+      			</joint>
+		</transmission>-->
 	</xacro:macro>
 	<xacro:wheel prefix="right" reflect="1" />

Commit message: Auto stash before merge of "master" and "origin/master"
State_publisher is working better, laser_scan launch file added

File: stiu_setup_tf/urdf/stiu.xacro (robot description, xacro)
@@ -5,4 +5,9 @@
 	 xmlns:xacro="http://playerstage.sourceforge.net/gazebo/xmlschema/#interface"
 	 name="stiu">
+	<xacro:property name="pi" value="3.1415926535897931" />
+  	<xacro:rplidar name="rplidar" parent="base_link" ros_topic="scan" update_rate="5" ray_count="1040" min_angle="0" max_angle="360">
+		<origin xyz="0 0 0.06" rpy="0 0 0"/>
+		<!-- <origin xyz="-0.1 0 0.420" rpy="3.1415 0 1.5707"/>-->
+	</xacro:rplidar>
 	<xacro:property name="width" value=".2" />
 	<xacro:property name="leglen" value=".6" />
@@ -11,5 +16,4 @@
 	<xacro:property name="baselen" value=".4" />
 	<xacro:property name="wheeldiam" value=".065" />
-	<xacro:property name="pi" value="3.1415" />
 	<xacro:macro name="default_inertial" params="mass">
 		<inertial>
@@ -83,5 +87,73 @@
       			</joint>
 		</transmission>-->
-	</xacro:macro>
+	 </xacro:macro>
+	<xacro:macro name="rplidar_model" params="name parent *origin">
+	      <joint name="${name}_joint" type="fixed">
+		<xacro:insert_block name="origin" />
+		<parent link="${parent}"/>
+		<!-- <child link="${name}_frame"/>-->
+		<child link="laser"/>
+	      </joint>
+	      <!-- <link name="${name}_frame">-->
+		<link name="laser">
+		<inertial>
+		  <mass value="0.270" />
+		  <origin xyz="0 0 0" rpy="0 0 0" />
+		  <inertia ixx="2.632e-4" ixy="0" ixz="0" iyy="2.632e-4" iyz="0" izz="1.62e-4" />
+		</inertial>
+		<visual>
+		  <origin xyz="0 0 0" rpy="0 0 0" />
+		  <geometry>
+		  <mesh filename="package://hector_sensors_description/meshes/hokuyo_utm30lx/hokuyo_utm_30lxTEST_SELF_FILTER.dae"/>
+		</geometry>
+		</visual>
+		<collision>
+		  <origin xyz="0 0 -0.0115" rpy="0 0 0" />
+		  <geometry>
+		  <box size="0.058 0.058 0.087" />
+		  <mesh filename="package://hector_sensors_description/meshes/hokuyo_utm30lx/hokuyo_utm_30lx.stl"/>
+		</geometry>
+		</collision>
+	      </link>
+	    </xacro:macro>
+	    <xacro:macro name="rplidar" params="name parent *origin ros_topic update_rate ray_count min_angle max_angle">
+	      <xacro:rplidar_model name="${name}" parent="${parent}">
+		<xacro:insert_block name="origin" />
+	      </xacro:rplidar_model>
+	      <!--<gazebo reference="${name}_frame">-->
+	      <gazebo reference="laser">
+		<sensor type="ray" name="${name}">
+		  <always_on>true</always_on>
+		  <update_rate>${update_rate}</update_rate>
+		  <pose>0 0 0 0 0 0</pose>
+		  <visualize>false</visualize>
+		  <ray>
+		    <scan>
+		      <horizontal>
+		        <samples>${ray_count}</samples>
+		        <resolution>1</resolution>
+		        <min_angle>${min_angle * pi/180}</min_angle>
+		        <max_angle>${max_angle * pi/180}</max_angle>
+		      </horizontal>
+		    </scan>
+		    <range>
+		      <min>0.2</min>
+		      <max>15.0</max>
+		      <resolution>0.01</resolution>
+		    </range>
+		    <noise>
+		      <type>gaussian</type>
+		      <mean>0.0</mean>
+		      <stddev>0.004</stddev>
+		    </noise>
+		  </ray>
+		  <plugin name="gazebo_ros_${name}_controller" filename="libgazebo_ros_laser.so">
+		    <topicName>${ros_topic}</topicName>
+		    <frameName>laser</frameName>
+		    <!--<frameName>${name}_frame</frameName>-->
+		  </plugin>
+		</sensor>
+	      </gazebo>
+	    </xacro:macro>
 	<xacro:wheel prefix="right" reflect="1" />
 	<xacro:wheel prefix="left" reflect="-1" />
